Commit message: angepasst auf neue Aufgabenstellung

File: assets/urdf/robot_without_gripper.urdf (robot description, URDF)
Before this commit: robot ur10e_cell, 18 links, 16 joints
Links:
- added link cylinder_link; visual cylinder length=0.2 radius=0.01
- added link tcp_link
Joints:
- added joint cylinder-tcp: type fixed, parent cylinder_link, child tcp_link, origin xyz=0.0 0.0 0.2 rpy=0 0 0
- added joint flange-tool0: type fixed, parent flange, child tool0, origin xyz=0 0 0 rpy=1.5707963267948966 0 1.5707963267948966
- added joint tool1: type fixed, parent tool0, child cylinder_link, origin xyz=0.0 0.0 0.0 rpy=0 0 3.141592653589793

Commit message: added more objects

File: assets/urdf/robot_without_gripper.urdf (robot description, URDF)
Before this commit: robot ur10e_cell, 20 links, 19 joints
Links:
- link cylinder_link: mass None -> 0.2; geometry collision cylinder length=0.1 radius=0.01; visual cylinder length=0.1 radius=0.01
