Commit message: changed goal size to 0.16m (max 9 objects per goal)

File: assets/objects/goals/goal_green.urdf (robot description, URDF)
Before this commit: robot rectangleexample, 5 links, 4 joints
Links:
- link bottom_border: geometry visual box size=0.16 0.001 0.001
- link left_border: geometry visual box size=0.001 0.162 0.001
- link right_border: geometry visual box size=0.001 0.162 0.001
- link top_border: geometry visual box size=0.16 0.001 0.001
Joints:
- joint bottom_border_joint: origin xyz=0 -0.0305 0 rpy=0 0 0 -> xyz=0 -0.0805 0 rpy=0 0 0
- joint left_border_joint: origin xyz=-0.0305 0 0 rpy=0 0 0 -> xyz=-0.0805 0 0 rpy=0 0 0
- joint right_border_joint: origin xyz=0.0305 0 0 rpy=0 0 0 -> xyz=0.0805 0 0 rpy=0 0 0
- joint top_border_joint: origin xyz=0 0.0305 0 rpy=0 0 0 -> xyz=0 0.0805 0 rpy=0 0 0

File: assets/objects/goals/goal_red.urdf (robot description, URDF)
Before this commit: robot rectangleexample, 5 links, 4 joints
Links:
- link bottom_border: geometry visual box size=0.16 0.001 0.001
- link left_border: geometry visual box size=0.001 0.162 0.001
- link right_border: geometry visual box size=0.001 0.162 0.001
- link top_border: geometry visual box size=0.16 0.001 0.001
Joints:
- joint bottom_border_joint: origin xyz=0 -0.0305 0 rpy=0 0 0 -> xyz=0 -0.0805 0 rpy=0 0 0
- joint left_border_joint: origin xyz=-0.0305 0 0 rpy=0 0 0 -> xyz=-0.0805 0 0 rpy=0 0 0
- joint right_border_joint: origin xyz=0.0305 0 0 rpy=0 0 0 -> xyz=0.0805 0 0 rpy=0 0 0
- joint top_border_joint: origin xyz=0 0.0305 0 rpy=0 0 0 -> xyz=0 0.0805 0 rpy=0 0 0
